Commit message: feat: 更新机器人模型配置，修改 URDF 文件路径并添加 RViz 配置文件

File: chapt6/chapt6_ws/src/fishbot_description/urdf/first_robot.urdf.xacro (robot description, xacro)
@@ -1,4 +1,11 @@
 <?xml version="1.0"?>
 <robot xmlns:xacro="http://www.ros.org/wiki/xacro" name="first_robot">
+    <!-- 定义材质，在 robot 级别 -->
+    <material name="blue">
+        <color rgba="0.1 0.1 1.0 0.5" />
+    </material>
+    <material name="black">
+        <color rgba="0 0 0 0.5" />
+    </material>
     <!-- 声明 base 模块 -->
     <xacro:macro name="base_link" params="length radius">
@@ -9,7 +16,5 @@
                     <cylinder length="${length}" radius="${length}" />
                 </geometry>
-                <material name="blue">
-                    <color rgba="0.1 0.1 1.0 0.5" />
-                </material>
+                <material name="blue"/>
             </visual>
         </link>
@@ -23,8 +28,6 @@
                     <box size="0.02 0.02 0.02" />
                 </geometry>
+                <material name="black"/>
             </visual>
-            <material name="black">
-                <color rgba="0 0 0 0.5" />
-            </material>
         </link>
         <joint name="${imu_name}_joint" type="fixed">
