Commit message: migrate(gazebo): migrate from Gazebo Classic to Gazebo Sim
将 fishbot 仿真环境从 Gazebo Classic 迁移到 Gazebo Sim (Ignition)，
以适配 ROS 2 Jazzy 和现代仿真工具链。

主要变更：
- launch 文件：使用 ros_gz_sim 替代 gazebo_ros
- ros2_control：使用 gz_ros2_control/GazeboSimSystem 硬件插件
- 插件库：libgazebo_ros2_control.so → libgz_ros2_control-system.so
- 移除 diff_drive 插件（由 ros2_control 处理）
- 移除传感器插件（使用 ros_gz_bridge 桥接）
- 更新 pixi.toml 依赖：添加 ros-jazzy-ros-gz-* 和 ros2-control 相关包

File: chapt6/chapt6_ws/src/fishbot_description/urdf/fishbot/fishbot.ros2_control.xacro (robot description, xacro)
@@ -4,5 +4,5 @@
     <ros2_control name="FishBotGazeboSystem" type="system">
             <hardware>
-                <plugin>gazebo_ros2_control/GazeboSystem</plugin>
+                <plugin>gz_ros2_control/GazeboSimSystem</plugin>
             </hardware>
             <joint name="left_wheel_joint">
@@ -34,5 +34,5 @@
         </ros2_control>
         <gazebo>
-        <plugin filename="libgazebo_ros2_control.so" name="gazebo_ros2_control">
+        <plugin filename="libgz_ros2_control-system.so" name="gz_ros2_control::GazeboSimROS2ControlPlugin">
             <parameters>$(find fishbot_description)/config/fishbot_ros2_controller.yaml</parameters>
             <ros>

File: chapt6/chapt6_ws/src/fishbot_description/urdf/fishbot/plugins/gazebo_control_plugin.xacro (robot description, xacro)
@@ -1,30 +1,6 @@
 <?xml version="1.0"?>
 <robot xmlns:xacro="http://www.ros.org/wiki/xacro">
+    <!-- Gazebo Sim uses ros2_control for diff drive, no separate plugin needed -->
     <xacro:macro name="gazebo_control_plugin">
-        <gazebo>
-            <plugin name='diff_drive' filename='libgazebo_ros_diff_drive.so'>
-                <ros>
-                    <namespace>/</namespace>
-                    <remapping>cmd_vel:=cmd_vel</remapping>
-                    <remapping>odom:=odom</remapping>
-                </ros>
-                <update_rate>30</update_rate>
-                <!-- wheels -->
-                <left_joint>left_wheel_joint</left_joint>
-                <right_joint>right_wheel_joint</right_joint>
-                <!-- kinematics -->
-                <wheel_separation>0.2</wheel_separation>
-                <wheel_diameter>0.064</wheel_diameter>
-                <!-- limits -->
-                <max_wheel_torque>20</max_wheel_torque>
-                <max_wheel_acceleration>1.0</max_wheel_acceleration>
-                <!-- output -->
-                <publish_odom>true</publish_odom>
-                <publish_odom_tf>true</publish_odom_tf>
-                <publish_wheel_tf>true</publish_wheel_tf>
-                <odometry_frame>odom</odometry_frame>
-                <robot_base_frame>base_footprint</robot_base_frame>
-            </plugin>
-        </gazebo>
-   </xacro:macro>
+    </xacro:macro>
 </robot>

File: chapt6/chapt6_ws/src/fishbot_description/urdf/fishbot/plugins/gazebo_sensor_plugin.xacro (robot description, xacro)
@@ -1,138 +1,6 @@
 <?xml version="1.0"?>
 <robot xmlns:xacro="http://www.ros.org/wiki/xacro">
+    <!-- Gazebo Sim uses ros_gz_bridge for sensor data, no plugins needed -->
     <xacro:macro name="gazebo_sensor_plugin">
-        <gazebo reference="laser_link">
-            <sensor name="laserscan" type="ray">
-                <plugin name="laserscan" filename="libgazebo_ros_ray_sensor.so">
-                    <ros>
-                        <namespace>/</namespace>
-                        <remapping>~/out:=scan</remapping>
-                    </ros>
-                    <output_type>sensor_msgs/LaserScan</output_type>
-                    <frame_name>laser_link</frame_name>
-                </plugin>
-                <always_on>true</always_on>
-                <visualize>true</visualize>
-                <update_rate>5</update_rate>
-                <pose>0 0 0 0 0 0</pose>
-								<!-- 激光传感器配置 -->
-                <ray>
-                    <!-- 设置扫描范围 -->
-                    <scan>
-                        <horizontal>
-                            <samples>360</samples>
-                            <resolution>1.000000</resolution>
-                            <min_angle>0.000000</min_angle>
-                            <max_angle>6.280000</max_angle>
-                        </horizontal>
-                    </scan>
-                    <!-- 设置扫描距离 -->
-                    <range>
-                        <min>0.120000</min>
-                        <max>8.0</max>
-                        <resolution>0.015000</resolution>
-                    </range>
-                    <!-- 设置噪声 -->
-                    <noise>
-                        <type>gaussian</type>
-                        <mean>0.0</mean>
-                        <stddev>0.01</stddev>
-                    </noise>
-                </ray>
-            </sensor>
-        </gazebo>
-<gazebo reference="imu_link">
-    <sensor name="imu_sensor" type="imu">
-        <plugin name="imu_plugin" filename="libgazebo_ros_imu_sensor.so">
-            <ros>
-                <namespace>/</namespace>
-                <remapping>~/out:=imu</remapping>
-            </ros>
-            <initial_orientation_as_reference>false</initial_orientation_as_reference>
-        </plugin>
-        <update_rate>100</update_rate>
-        <always_on>true</always_on>
-        <!-- 六轴噪声设置 -->
-        <imu>
-            <angular_velocity>
-                <x>
-                    <noise type="gaussian">
-                        <mean>0.0</mean>
-                        <stddev>2e-4</stddev>
-                        <bias_mean>0.0000075</bias_mean>
-                        <bias_stddev>0.0000008</bias_stddev>
-                    </noise>
-                </x>
-                <y>
-                    <noise type="gaussian">
-                        <mean>0.0</mean>
-                        <stddev>2e-4</stddev>
-                        <bias_mean>0.0000075</bias_mean>
-                        <bias_stddev>0.0000008</bias_stddev>
-                    </noise>
-                </y>
-                <z>
-                    <noise type="gaussian">
-                        <mean>0.0</mean>
-                        <stddev>2e-4</stddev>
-                        <bias_mean>0.0000075</bias_mean>
-                        <bias_stddev>0.0000008</bias_stddev>
-                    </noise>
-                </z>
-            </angular_velocity>
-            <linear_acceleration>
-                <x>
-                    <noise type="gaussian">
-                        <mean>0.0</mean>
-                        <stddev>1.7e-2</stddev>
-                        <bias_mean>0.1</bias_mean>
-                        <bias_stddev>0.001</bias_stddev>
-                    </noise>
-                </x>
-                <y>
-                    <noise type="gaussian">
-                        <mean>0.0</mean>
-                        <stddev>1.7e-2</stddev>
-                        <bias_mean>0.1</bias_mean>
-                        <bias_stddev>0.001</bias_stddev>
-                    </noise>
-                </y>
-                <z>
-                    <noise type="gaussian">
-                        <mean>0.0</mean>
-                        <stddev>1.7e-2</stddev>
-                        <bias_mean>0.1</bias_mean>
-                        <bias_stddev>0.001</bias_stddev>
-                    </noise>
-                </z>
-            </linear_acceleration>
-        </imu>
-    </sensor>
-</gazebo>
     </xacro:macro>
-<gazebo reference="camera_link">
-    <sensor type="depth" name="camera_sensor">
-        <plugin name="depth_camera" filename="libgazebo_ros_camera.so">
-            <frame_name>camera_optical_link</frame_name>
-        </plugin>
-        <always_on>true</always_on>
-        <update_rate>10</update_rate>
-        <camera name="camera">
-            <horizontal_fov>1.5009831567</horizontal_fov>
-            <image>
-                <width>800</width>
-                <height>600</height>
-                <format>R8G8B8</format>
-            </image>
-            <distortion>
-                <k1>0.0</k1>
-                <k2>0.0</k2>
-                <k3>0.0</k3>
-                <p1>0.0</p1>
-                <p2>0.0</p2>
-                <center>0.5 0.5</center>
-            </distortion>
-        </camera>
-    </sensor>
-</gazebo>
 </robot>
